File: hardware/pnb-1/sch/pnb-1.kicad_sch (KiCad schematic)
At the start: 33 parts, among them J1 USB-C 16P, J3 DTR 2x6, J4 UART 1x4, SW1 BOOT, SW2 RESET, U1 ESP32-S3-MINI-1-N8, U2 AMS1117-3.3, U3 SCD41-D-R2, U4 BH1750FVI-TR

Commit message: fix(pcb): correct sensor land pattern and release gates
Parts:
- removed C9: 22uF tantalum, artera:CASE-A_3216, symbol artera:CL21A226MAQNNNE
- added C9: 22uF tantalum, artera:CASE-A_3216, symbol artera:TAJA226K010RNJ
- J3: value DTR 2x6 -> DTR 2x6 DNP; now not fitted; now left out of the parts list
Connections:
- net 3V3: now also C9.1
- net GND: now also C9.2; no longer U3.21 (GND)
